Commit message: Synapses Done

File: body.urdf (robot description, URDF)
Before this commit: robot robot, 3 links, 2 joints
Joints:
- removed joint FrontLeg_Torso
- added joint Torso_FrontLeg: type revolute, parent FrontLeg, child Torso, origin xyz=1.0 0.5 1.0 rpy=0 0 0, axis 0 1 0, limit lower=-3.14159 upper=3.14159 effort=0.0 velocity=0.0
