Commit message: Finished Building Bot

File: Body.urdf (robot description, URDF)
Before this commit: robot robot, 9 links, 8 joints
Links:
- removed link BackLeg
- removed link BackLeg2
- removed link FrontLeg
- removed link FrontLeg2
- removed link LeftLeg
- removed link LeftLeg2
- removed link RightLeg
- removed link RightLeg2
- added link Leg1A, mass 10; collision box size=0.2 0.2 1.0; visual box size=0.2 0.2 1.0
- added link Leg1B, mass 10; collision box size=0.2 0.2 1.0; visual box size=0.2 0.2 1.0
- added link Leg2A, mass 10; collision box size=0.2 0.2 1.0; visual box size=0.2 0.2 1.0
- added link Leg2B, mass 10; collision box size=0.2 0.2 1.0; visual box size=0.2 0.2 1.0
- added link Leg3A, mass 10; collision box size=0.2 0.2 1.0; visual box size=0.2 0.2 1.0
- added link Leg3B, mass 10; collision box size=0.2 0.2 1.0; visual box size=0.2 0.2 1.0
- added link Leg4A, mass 10; collision box size=0.2 0.2 1.0; visual box size=0.2 0.2 1.0
- added link Leg4B, mass 10; collision box size=0.2 0.2 1.0; visual box size=0.2 0.2 1.0
- added link Rod1, mass 10; collision box size=0.2 0.2 0.6; visual box size=0.2 0.2 0.6
- added link Rod2, mass 10; collision box size=0.6 0.2 0.2; visual box size=0.6 0.2 0.2
- link Torso: mass 1 -> 10; geometry collision box size=1.8 1.0 0.5; visual box size=1.8 1.0 0.5
Joints:
- removed joint Torso_BackLeg
- removed joint Torso_BackLeg2
- removed joint Torso_FrontLeg
- removed joint Torso_FrontLeg2
- removed joint Torso_LeftLeg
- removed joint Torso_LeftLeg2
- removed joint Torso_RightLeg
- removed joint Torso_RightLeg2
- added joint Leg1A_Leg1B: type revolute, parent Leg1A, child Leg1B, origin xyz=0.0 0.0 -1.0 rpy=0 0 0, axis 0 1 0, limit lower=-3.14159 upper=3.14159 effort=0.0 velocity=0.0
- added joint Leg2A_Leg2B: type revolute, parent Leg2A, child Leg2B, origin xyz=0.0 0.0 -1.0 rpy=0 0 0, axis 0 1 0, limit lower=-3.14159 upper=3.14159 effort=0.0 velocity=0.0
- added joint Leg3A_Leg3B: type revolute, parent Leg3A, child Leg3B, origin xyz=0.0 0 -1.0 rpy=0 0 0, axis 0 1 0, limit lower=-3.14159 upper=3.14159 effort=0.0 velocity=0.0
- added joint Leg4A_Leg4B: type revolute, parent Leg4A, child Leg4B, origin xyz=0.0 0.0 -1.0 rpy=0 0 0, axis 0 1 0, limit lower=-3.14159 upper=3.14159 effort=0.0 velocity=0.0
- added joint Rod1_Rod2: type revolute, parent Rod1, child Rod2, origin xyz=0.0 0.0 0.6 rpy=0 0 0, axis 0 1 0, limit lower=-3.14159 upper=3.14159 effort=0.0 velocity=0.0
- added joint Torso_Leg1A: type revolute, parent Torso, child Leg1A, origin xyz=0.5 0.5 2.0 rpy=0 0 0, axis 1 1 0, limit lower=-3.14159 upper=3.14159 effort=0.0 velocity=0.0
- added joint Torso_Leg2A: type revolute, parent Torso, child Leg2A, origin xyz=-0.5 0.5 2.0 rpy=0 0 0, axis 1 1 0, limit lower=-3.14159 upper=3.14159 effort=0.0 velocity=0.0
- added joint Torso_Leg3A: type revolute, parent Torso, child Leg3A, origin xyz=0.5 -0.5 2.0 rpy=0 0 0, axis 1 1 0, limit lower=-3.14159 upper=3.14159 effort=0.0 velocity=0.0
- added joint Torso_Leg4A: type revolute, parent Torso, child Leg4A, origin xyz=-0.5 -0.5 2.0 rpy=0 0 0, axis 1 1 0, limit lower=-3.14159 upper=3.14159 effort=0.0 velocity=0.0
- added joint Torso_Rod: type revolute, parent Torso, child Rod1, origin xyz=0.5 0.0 2.25 rpy=0 0 0, axis 0 1 0, limit lower=-3.14159 upper=3.14159 effort=0.0 velocity=0.0

Commit message: Updated Code

File: Body.urdf (robot description, URDF)
Before this commit: robot robot, 11 links, 10 joints
Links:
- link Leg1A: geometry collision box size=0.3 0.3 1.0; visual box size=0.3 0.3 1.0
- link Leg1B: geometry collision box size=0.3 0.3 1.0; visual box size=0.3 0.3 1.0
- link Leg2A: geometry collision box size=0.3 0.3 1.0; visual box size=0.3 0.3 1.0
- link Leg2B: geometry collision box size=0.3 0.3 1.0; visual box size=0.3 0.3 1.0
- link Leg3A: geometry collision box size=0.3 0.3 1.0; visual box size=0.3 0.3 1.0
- link Leg3B: geometry collision box size=0.3 0.3 1.0; visual box size=0.3 0.3 1.0
- link Leg4A: geometry collision box size=0.3 0.3 1.0; visual box size=0.3 0.3 1.0
- link Leg4B: geometry collision box size=0.3 0.3 1.0; visual box size=0.3 0.3 1.0
- link Rod1: geometry collision box size=0.3 0.3 0.6; visual box size=0.3 0.3 0.6
- link Rod2: geometry collision box size=0.6 0.3 0.3; visual box size=0.6 0.3 0.3
- link Torso: geometry collision box size=1.7 1.0 0.5; visual box size=1.7 1.0 0.5
Joints:
- removed joint Torso_Rod
- added joint Torso_Rod1: type revolute, parent Torso, child Rod1, origin xyz=0.5 0.0 2.25 rpy=0 0 0, axis 0 1 0, limit lower=-3.14159 upper=3.14159 effort=0.0 velocity=0.0

Commit message: Code now works on uvm w3 servers

File: Body.urdf (robot description, URDF)
Before this commit: robot robot, 11 links, 10 joints
Links:
- link Leg1A: mass 10 -> 7
- link Leg1B: mass 10 -> 7; geometry collision box size=0.3 0.3 0.7; visual box size=0.3 0.3 0.7
- link Leg2A: mass 10 -> 7
- link Leg2B: mass 10 -> 7; geometry collision box size=0.3 0.3 0.7; visual box size=0.3 0.3 0.7
- link Leg3A: mass 10 -> 7
- link Leg3B: mass 10 -> 7; geometry collision box size=0.3 0.3 0.7; visual box size=0.3 0.3 0.7
- link Leg4A: mass 10 -> 7
- link Leg4B: mass 10 -> 7; geometry collision box size=0.3 0.3 0.7; visual box size=0.3 0.3 0.7
- link Rod1: mass 10 -> 7
- link Rod2: mass 10 -> 7
- link Torso: mass 10 -> 7
Joints:
- joint Leg1A_Leg1B: origin xyz=0.0 0.0 -1.0 rpy=0 0 0 -> xyz=0.0 0.0 -0.7 rpy=0 0 0
- joint Leg2A_Leg2B: origin xyz=0.0 0.0 -1.0 rpy=0 0 0 -> xyz=0.0 0.0 -0.7 rpy=0 0 0
- joint Leg3A_Leg3B: origin xyz=0.0 0 -1.0 rpy=0 0 0 -> xyz=0.0 0 -0.7 rpy=0 0 0
- joint Leg4A_Leg4B: origin xyz=0.0 0.0 -1.0 rpy=0 0 0 -> xyz=0.0 0.0 -0.7 rpy=0 0 0
- joint Torso_Leg1A: origin xyz=0.5 0.5 2.0 rpy=0 0 0 -> xyz=0.5 0.6 2.0 rpy=0 0 0
- joint Torso_Leg2A: origin xyz=-0.5 0.5 2.0 rpy=0 0 0 -> xyz=-0.5 0.6 2.0 rpy=0 0 0
- joint Torso_Leg3A: origin xyz=0.5 -0.5 2.0 rpy=0 0 0 -> xyz=0.5 -0.6 2.0 rpy=0 0 0
- joint Torso_Leg4A: origin xyz=-0.5 -0.5 2.0 rpy=0 0 0 -> xyz=-0.5 -0.6 2.0 rpy=0 0 0

Commit message: Made it more like the MIT Spot dog

File: Body.urdf (robot description, URDF)
Before this commit: robot robot, 11 links, 10 joints
Links:
- removed link Rod1
- removed link Rod2
- added link Foot1, mass 7; collision sphere radius=0.2; visual sphere radius=0.2
- added link Foot2, mass 7; collision sphere radius=0.2; visual sphere radius=0.2
- added link Foot3, mass 7; collision sphere radius=0.2; visual sphere radius=0.2
- added link Foot4, mass 7; collision sphere radius=0.2; visual sphere radius=0.2
- link Leg1A: geometry collision box size=0.25 0.23 1.1; visual box size=0.25 0.23 1.1
- link Leg1B: geometry collision box size=0.2 0.22 0.8; visual box size=0.2 0.22 0.8
- link Leg2A: geometry collision box size=0.25 0.23 1.1; visual box size=0.25 0.23 1.1
- link Leg2B: geometry collision box size=0.2 0.22 0.8; visual box size=0.2 0.22 0.8
- link Leg3A: geometry collision box size=0.25 0.23 1.1; visual box size=0.25 0.23 1.1
- link Leg3B: geometry collision box size=0.2 0.22 0.8; visual box size=0.2 0.22 0.8
- link Leg4A: geometry collision box size=0.25 0.23 1.1; visual box size=0.25 0.23 1.1
- link Leg4B: geometry collision box size=0.2 0.22 0.8; visual box size=0.2 0.22 0.8
- link Torso: geometry collision box size=2.5 1.0 0.5; visual box size=2.5 1.0 0.5
Joints:
- removed joint Rod1_Rod2
- removed joint Torso_Rod1
- added joint Leg1B_Foot1: type fixed, parent Leg1B, child Foot1, origin xyz=0.0 0.0 0.0 rpy=0 0 0, axis 0 0 0, limit lower=-3.14159 upper=3.14159 effort=0.0 velocity=0.0
- added joint Leg2B_Foot2: type fixed, parent Leg2B, child Foot2, origin xyz=0.0 0.0 0.0 rpy=0 0 0, axis 0 0 0, limit lower=-3.14159 upper=3.14159 effort=0.0 velocity=0.0
- added joint Leg3B_Foot3: type fixed, parent Leg3B, child Foot3, origin xyz=0.0 0.0 0.0 rpy=0 0 0, axis 0 0 0, limit lower=-3.14159 upper=3.14159 effort=0.0 velocity=0.0
- added joint Leg4B_Foot4: type fixed, parent Leg4B, child Foot4, origin xyz=0.0 0.0 0.0 rpy=0 0 0, axis 0 0 0, limit lower=-3.14159 upper=3.14159 effort=0.0 velocity=0.0
- joint Leg1A_Leg1B: origin xyz=0.0 0.0 -0.7 rpy=0 0 0 -> xyz=-0.1 0.0 -0.7 rpy=0 0 0
- joint Leg2A_Leg2B: origin xyz=0.0 0.0 -0.7 rpy=0 0 0 -> xyz=-0.1 0.0 -0.7 rpy=0 0 0
- joint Leg3A_Leg3B: origin xyz=0.0 0 -0.7 rpy=0 0 0 -> xyz=-0.1 0.0 -0.7 rpy=0 0 0
- joint Leg4A_Leg4B: origin xyz=0.0 0.0 -0.7 rpy=0 0 0 -> xyz=-0.1 0.0 -0.7 rpy=0 0 0
- joint Torso_Leg1A: origin xyz=0.5 0.6 2.0 rpy=0 0 0 -> xyz=0.725 0.6 2.1 rpy=0 0 0
- joint Torso_Leg2A: origin xyz=-0.5 0.6 2.0 rpy=0 0 0 -> xyz=-0.725 0.6 2.1 rpy=0 0 0
- joint Torso_Leg3A: origin xyz=0.5 -0.6 2.0 rpy=0 0 0 -> xyz=0.725 -0.6 2.1 rpy=0 0 0
- joint Torso_Leg4A: origin xyz=-0.5 -0.6 2.0 rpy=0 0 0 -> xyz=-0.725 -0.6 2.1 rpy=0 0 0

Commit message: Changed bot so angle works, starts on ground

File: Body.urdf (robot description, URDF)
Before this commit: robot robot, 13 links, 12 joints
Links:
- link Foot1: mass 7 -> 5
- link Foot2: mass 7 -> 5
- link Foot3: mass 7 -> 5
- link Foot4: mass 7 -> 5
- link Leg1A: mass 7 -> 5
- link Leg1B: mass 7 -> 5
- link Leg2A: mass 7 -> 5
- link Leg2B: mass 7 -> 5
- link Leg3A: mass 7 -> 5
- link Leg3B: mass 7 -> 5
- link Leg4A: mass 7 -> 5
- link Leg4B: mass 7 -> 5
- link Torso: mass 7 -> 5
Joints:
- joint Leg1A_Leg1B: origin xyz=-0.1 0.0 -0.7 rpy=0 0 0 -> xyz=0.0 0.0 -0.9 rpy=0 0 0
- joint Leg1B_Foot1: origin xyz=0.0 0.0 0.0 rpy=0 0 0 -> xyz=0.95 0.0 0.0 rpy=0 0 0
- joint Leg2A_Leg2B: origin xyz=-0.1 0.0 -0.7 rpy=0 0 0 -> xyz=0.0 0.0 -0.9 rpy=0 0 0
- joint Leg2B_Foot2: origin xyz=0.0 0.0 0.0 rpy=0 0 0 -> xyz=0.95 0.0 0.0 rpy=0 0 0
- joint Leg3A_Leg3B: origin xyz=-0.1 0.0 -0.7 rpy=0 0 0 -> xyz=0.0 0.0 -0.9 rpy=0 0 0
- joint Leg3B_Foot3: origin xyz=0.0 0.0 0.0 rpy=0 0 0 -> xyz=0.95 0.0 0.0 rpy=0 0 0
- joint Leg4A_Leg4B: origin xyz=-0.1 0.0 -0.7 rpy=0 0 0 -> xyz=0.0 0.0 -0.9 rpy=0 0 0
- joint Leg4B_Foot4: origin xyz=0.0 0.0 0.0 rpy=0 0 0 -> xyz=0.95 0.0 0.0 rpy=0 0 0

Commit message: Working bot with altered fitness function

File: Body.urdf (robot description, URDF)
Before this commit: robot robot, 13 links, 12 joints
Links:
- link Foot1: mass 5 -> 4; geometry collision sphere radius=0.18; visual sphere radius=0.18
- link Foot2: mass 5 -> 4; geometry collision sphere radius=0.18; visual sphere radius=0.18
- link Foot3: mass 5 -> 4; geometry collision sphere radius=0.18; visual sphere radius=0.18
- link Foot4: mass 5 -> 4; geometry collision sphere radius=0.18; visual sphere radius=0.18
- link Leg1A: mass 5 -> 4
- link Leg1B: mass 5 -> 4; geometry collision box size=0.2 0.22 1.1; visual box size=0.2 0.22 1.1
- link Leg2A: mass 5 -> 4
- link Leg2B: mass 5 -> 4; geometry collision box size=0.2 0.22 1.1; visual box size=0.2 0.22 1.1
- link Leg3A: mass 5 -> 4
- link Leg3B: mass 5 -> 4; geometry collision box size=0.2 0.22 1.1; visual box size=0.2 0.22 1.1
- link Leg4A: mass 5 -> 4
- link Leg4B: mass 5 -> 4; geometry collision box size=0.2 0.22 1.1; visual box size=0.2 0.22 1.1
- link Torso: mass 5 -> 4; geometry collision box size=2.5 1.1 0.5; visual box size=2.5 1.1 0.5
Joints:
- joint Leg1A_Leg1B: origin xyz=0.0 0.0 -0.9 rpy=0 0 0 -> xyz=-0.52 0.0 -0.92 rpy=0 0 0
- joint Leg1B_Foot1: origin xyz=0.95 0.0 0.0 rpy=0 0 0 -> xyz=0.55 0.0 -0.68 rpy=0 0 0
- joint Leg2A_Leg2B: origin xyz=0.0 0.0 -0.9 rpy=0 0 0 -> xyz=-0.52 0.0 -0.92 rpy=0 0 0
- joint Leg2B_Foot2: origin xyz=0.95 0.0 0.0 rpy=0 0 0 -> xyz=0.55 0.0 -0.68 rpy=0 0 0
- joint Leg3A_Leg3B: origin xyz=0.0 0.0 -0.9 rpy=0 0 0 -> xyz=-0.52 0.0 -0.92 rpy=0 0 0
- joint Leg3B_Foot3: origin xyz=0.95 0.0 0.0 rpy=0 0 0 -> xyz=0.55 0.0 -0.68 rpy=0 0 0
- joint Leg4A_Leg4B: origin xyz=0.0 0.0 -0.9 rpy=0 0 0 -> xyz=-0.52 0.0 -0.92 rpy=0 0 0
- joint Leg4B_Foot4: origin xyz=0.95 0.0 0.0 rpy=0 0 0 -> xyz=0.55 0.0 -0.68 rpy=0 0 0
- joint Torso_Leg1A: axis 1 1 0 -> 0 1 0
- joint Torso_Leg2A: axis 1 1 0 -> 0 1 0
- joint Torso_Leg3A: axis 1 1 0 -> 0 1 0
- joint Torso_Leg4A: axis 1 1 0 -> 0 1 0

Commit message: Working final bot

File: Body.urdf (robot description, URDF)
Before this commit: robot robot, 13 links, 12 joints
Links:
- link Foot1: mass 4 -> 1; geometry collision sphere radius=0.16; visual sphere radius=0.16
- link Foot2: mass 4 -> 1; geometry collision sphere radius=0.16; visual sphere radius=0.16
- link Foot3: mass 4 -> 1; geometry collision sphere radius=0.16; visual sphere radius=0.16
- link Foot4: mass 4 -> 1; geometry collision sphere radius=0.16; visual sphere radius=0.16
- link Leg1A: mass 4 -> 1; geometry collision box size=0.25 0.23 1; visual box size=0.25 0.23 1
- link Leg1B: mass 4 -> 1; geometry collision box size=0.2 0.22 1; visual box size=0.2 0.22 1
- link Leg2A: mass 4 -> 1; geometry collision box size=0.25 0.23 1; visual box size=0.25 0.23 1
- link Leg2B: mass 4 -> 1; geometry collision box size=0.2 0.22 1; visual box size=0.2 0.22 1
- link Leg3A: mass 4 -> 1; geometry collision box size=0.25 0.23 1; visual box size=0.25 0.23 1
- link Leg3B: mass 4 -> 1; geometry collision box size=0.2 0.22 1; visual box size=0.2 0.22 1
- link Leg4A: mass 4 -> 1; geometry collision box size=0.25 0.23 1; visual box size=0.25 0.23 1
- link Leg4B: mass 4 -> 1; geometry collision box size=0.2 0.22 1; visual box size=0.2 0.22 1
- link Torso: mass 4 -> 1; geometry collision box size=2.4 1.0 0.55; visual box size=2.4 1.0 0.55
Joints:
- joint Torso_Leg1A: origin xyz=0.725 0.6 2.1 rpy=0 0 0 -> xyz=0.7 0.6 2.3 rpy=0 0 0
- joint Torso_Leg2A: origin xyz=-0.725 0.6 2.1 rpy=0 0 0 -> xyz=-0.7 0.6 2.3 rpy=0 0 0
- joint Torso_Leg3A: origin xyz=0.725 -0.6 2.1 rpy=0 0 0 -> xyz=0.7 -0.6 2.3 rpy=0 0 0
- joint Torso_Leg4A: origin xyz=-0.725 -0.6 2.1 rpy=0 0 0 -> xyz=-0.7 -0.6 2.3 rpy=0 0 0

Commit message: Half of size of original bot

File: Body.urdf (robot description, URDF)
Before this commit: robot robot, 13 links, 12 joints
Links:
- link Foot1: mass 1 -> 2; geometry collision sphere radius=0.08; visual sphere radius=0.08
- link Foot2: mass 1 -> 2; geometry collision sphere radius=0.08; visual sphere radius=0.08
- link Foot3: mass 1 -> 2; geometry collision sphere radius=0.08; visual sphere radius=0.08
- link Foot4: mass 1 -> 2; geometry collision sphere radius=0.08; visual sphere radius=0.08
- link Leg1A: mass 1 -> 2; geometry collision box size=0.125 0.115 0.5; visual box size=0.125 0.115 0.5
- link Leg1B: mass 1 -> 2; geometry collision box size=0.1 0.11 0.5; visual box size=0.1 0.11 0.5
- link Leg2A: mass 1 -> 2; geometry collision box size=0.125 0.115 0.5; visual box size=0.125 0.115 0.5
- link Leg2B: mass 1 -> 2; geometry collision box size=0.1 0.11 0.5; visual box size=0.1 0.11 0.5
- link Leg3A: mass 1 -> 2; geometry collision box size=0.125 0.115 0.5; visual box size=0.125 0.115 0.5
- link Leg3B: mass 1 -> 2; geometry collision box size=0.1 0.11 0.5; visual box size=0.1 0.11 0.5
- link Leg4A: mass 1 -> 2; geometry collision box size=0.125 0.115 0.5; visual box size=0.125 0.115 0.5
- link Leg4B: mass 1 -> 2; geometry collision box size=0.1 0.11 0.5; visual box size=0.1 0.11 0.5
- link Torso: mass 1 -> 2; geometry collision box size=1.2 0.5 0.275; visual box size=1.2 0.5 0.275
Joints:
- joint Leg1A_Leg1B: origin xyz=-0.52 0.0 -0.92 rpy=0 0 0 -> xyz=-0.26 0.0 -0.46 rpy=0 0 0
- joint Leg1B_Foot1: origin xyz=0.55 0.0 -0.68 rpy=0 0 0 -> xyz=0.275 0.0 -0.34 rpy=0 0 0
- joint Leg2A_Leg2B: origin xyz=-0.52 0.0 -0.92 rpy=0 0 0 -> xyz=-0.26 0.0 -0.46 rpy=0 0 0
- joint Leg2B_Foot2: origin xyz=0.55 0.0 -0.68 rpy=0 0 0 -> xyz=0.275 0.0 -0.34 rpy=0 0 0
- joint Leg3A_Leg3B: origin xyz=-0.52 0.0 -0.92 rpy=0 0 0 -> xyz=-0.26 0.0 -0.46 rpy=0 0 0
- joint Leg3B_Foot3: origin xyz=0.55 0.0 -0.68 rpy=0 0 0 -> xyz=0.275 0.0 -0.34 rpy=0 0 0
- joint Leg4A_Leg4B: origin xyz=-0.52 0.0 -0.92 rpy=0 0 0 -> xyz=-0.26 0.0 -0.46 rpy=0 0 0
- joint Leg4B_Foot4: origin xyz=0.55 0.0 -0.68 rpy=0 0 0 -> xyz=0.275 0.0 -0.34 rpy=0 0 0
- joint Torso_Leg1A: origin xyz=0.7 0.6 2.3 rpy=0 0 0 -> xyz=0.35 0.3 1.15 rpy=0 0 0
- joint Torso_Leg2A: origin xyz=-0.7 0.6 2.3 rpy=0 0 0 -> xyz=-0.35 0.3 1.15 rpy=0 0 0
- joint Torso_Leg3A: origin xyz=0.7 -0.6 2.3 rpy=0 0 0 -> xyz=0.35 -0.3 1.15 rpy=0 0 0
- joint Torso_Leg4A: origin xyz=-0.7 -0.6 2.3 rpy=0 0 0 -> xyz=-0.35 -0.3 1.15 rpy=0 0 0

Commit message: Update to compare with the hidden neuron bot

File: Body.urdf (robot description, URDF)
Before this commit: robot robot, 13 links, 12 joints
Links:
- link Foot1: geometry collision sphere radius=0.08; visual sphere radius=0.08
- link Foot2: geometry collision sphere radius=0.08; visual sphere radius=0.08
- link Foot3: geometry collision sphere radius=0.08; visual sphere radius=0.08
- link Foot4: geometry collision sphere radius=0.08; visual sphere radius=0.08
- link Leg1A: geometry collision box size=0.125 0.115 0.5; visual box size=0.125 0.115 0.5
- link Leg1B: geometry collision box size=0.1 0.11 0.5; visual box size=0.1 0.11 0.5
- link Leg2A: geometry collision box size=0.125 0.115 0.5; visual box size=0.125 0.115 0.5
- link Leg2B: geometry collision box size=0.1 0.11 0.5; visual box size=0.1 0.11 0.5
- link Leg3A: geometry collision box size=0.125 0.115 0.5; visual box size=0.125 0.115 0.5
- link Leg3B: geometry collision box size=0.1 0.11 0.5; visual box size=0.1 0.11 0.5
- link Leg4A: geometry collision box size=0.125 0.115 0.5; visual box size=0.125 0.115 0.5
- link Leg4B: geometry collision box size=0.1 0.11 0.5; visual box size=0.1 0.11 0.5
- link Torso: geometry collision box size=1.2 0.5 0.275; visual box size=1.2 0.5 0.275
Joints:
- joint Leg1A_Leg1B: origin xyz=-0.52 0.0 -0.92 rpy=0 0 0 -> xyz=-0.26 0.0 -0.46 rpy=0 0 0
- joint Leg1B_Foot1: origin xyz=0.55 0.0 -0.68 rpy=0 0 0 -> xyz=0.275 0.0 -0.34 rpy=0 0 0
- joint Leg2A_Leg2B: origin xyz=-0.52 0.0 -0.92 rpy=0 0 0 -> xyz=-0.26 0.0 -0.46 rpy=0 0 0
- joint Leg2B_Foot2: origin xyz=0.55 0.0 -0.68 rpy=0 0 0 -> xyz=0.275 0.0 -0.34 rpy=0 0 0
- joint Leg3A_Leg3B: origin xyz=-0.52 0.0 -0.92 rpy=0 0 0 -> xyz=-0.26 0.0 -0.46 rpy=0 0 0
- joint Leg3B_Foot3: origin xyz=0.55 0.0 -0.68 rpy=0 0 0 -> xyz=0.275 0.0 -0.34 rpy=0 0 0
- joint Leg4A_Leg4B: origin xyz=-0.52 0.0 -0.92 rpy=0 0 0 -> xyz=-0.26 0.0 -0.46 rpy=0 0 0
- joint Leg4B_Foot4: origin xyz=0.55 0.0 -0.68 rpy=0 0 0 -> xyz=0.275 0.0 -0.34 rpy=0 0 0
- joint Torso_Leg1A: origin xyz=0.7 0.6 2.3 rpy=0 0 0 -> xyz=0.35 0.3 1.15 rpy=0 0 0
- joint Torso_Leg2A: origin xyz=-0.7 0.6 2.3 rpy=0 0 0 -> xyz=-0.35 0.3 1.15 rpy=0 0 0
- joint Torso_Leg3A: origin xyz=0.7 -0.6 2.3 rpy=0 0 0 -> xyz=0.35 -0.3 1.15 rpy=0 0 0
- joint Torso_Leg4A: origin xyz=-0.7 -0.6 2.3 rpy=0 0 0 -> xyz=-0.35 -0.3 1.15 rpy=0 0 0
